Commit message: Simulated Driving + Camera

File: description/robot.urdf.xacro (robot description, xacro)
@@ -2,3 +2,5 @@
 <robot xmlns:xacro="http://www.ros.org/wiki/xacro"  name="robot">
     <xacro:include filename="robot_core.xacro"/>
+    <xacro:include filename="gazebo_control.xacro" />
+    <xacro:include filename="camera.xacro" />
 </robot>

File: description/robot_core.xacro (robot description, xacro)
@@ -25,5 +25,5 @@
     <link name="chassis">
         <visual>
-            <origin xyz="0.085 0.0 0.02995"/>
+            <origin xyz="0.085 0.0 0.029"/>
             <geometry>
                 <box size="0.17 0.095 0.058"/>
@@ -32,5 +32,5 @@
         </visual>
         <collision>
-            <origin xyz="0.085 0.0 0.02995"/>
+            <origin xyz="0.085 0.0 0.029"/>
             <geometry>
                 <box size="0.17 0.095 0.058"/>
@@ -41,4 +41,7 @@
         </xacro:inertial_box>
     </link>
+    <gazebo reference="chassis">
+        <material>Gazebo/White</material>
+    </gazebo>
     <!-- LEFT FRONT WHEEL LINK -->
     <joint name="left_front_wheel_joint" type="continuous">
@@ -48,5 +51,85 @@
         <axis xyz="0.0 0.0 1.0" rpy="0.0 0.0 0.0"/>
     </joint>
-   <link name="left_front_wheel">
+    <link name="left_front_wheel">
+        <visual>
+            <geometry>
+                <cylinder radius="0.048" length="0.019"/>
+                <material name="blue"/>
+            </geometry>
+        </visual>
+        <collision>
+            <geometry>
+                <cylinder radius="0.048" length="0.019"/>
+            </geometry>
+        </collision>
+        <xacro:inertial_cylinder mass="0.1" length="0.019" radius="0.048">
+            <origin xyz="0 0 0" rpy="0 0 0" />
+        </xacro:inertial_cylinder>
+    </link>
+    <gazebo reference="left_front_wheel">
+        <material>Gazebo/Blue</material>
+    </gazebo>
+    <!-- LEFT REAR WHEEL LINK -->
+    <joint name="left_rear_wheel_joint" type="fixed">
+        <parent link="base_link"/>
+        <child link="left_rear_wheel"/>
+        <origin xyz="-0.05 0.058 0.025" rpy="-${pi/2} 0.0 0.0"/>
+        <axis xyz="0.0 0.0 1.0"/>
+    </joint>
+    <link name="left_rear_wheel">
+        <visual>
+            <geometry>
+                <cylinder radius="0.048" length="0.019"/>
+                <material name="blue"/>
+            </geometry>
+        </visual>
+        <collision>
+            <geometry>
+                <cylinder radius="0.048" length="0.019"/>
+            </geometry>
+        </collision>
+        <xacro:inertial_cylinder mass="0.1" length="0.019" radius="0.048">
+            <origin xyz="0 0 0" rpy="0 0 0" />
+        </xacro:inertial_cylinder>
+    </link>
+    <gazebo reference="left_rear_wheel">
+        <material>Gazebo/Blue</material>
+        <mu1 value="0.001"/>
+    </gazebo>
+    <!-- RIGHT FRONT WHEEL LINK -->
+    <joint name="right_front_wheel_joint" type="fixed">
+        <parent link="base_link"/>
+        <child link="right_front_wheel"/>
+        <origin xyz="0.05 -0.058 0.025" rpy="${pi/2} 0.0 0.0"/>
+        <axis xyz="0.0 0.0 -1.0"/>
+    </joint>
+    <link name="right_front_wheel">
+        <visual>
+            <geometry>
+                <cylinder radius="0.048" length="0.019"/>
+                <material name="blue"/>
+            </geometry>
+        </visual>
+        <collision>
+            <geometry>
+                <cylinder radius="0.048" length="0.019"/>
+            </geometry>
+        </collision>
+        <xacro:inertial_cylinder mass="0.1" length="0.019" radius="0.048">
+            <origin xyz="0 0 0" rpy="0 0 0" />
+        </xacro:inertial_cylinder>
+    </link>
+    <gazebo reference="right_front_wheel">
+        <material>Gazebo/Blue</material>
+        <mu1 value="0.001"/>
+    </gazebo>
+   <!-- RIGHT REAR WHEEL LINK -->
+    <joint name="right_rear_wheel_joint" type="continuous">
+        <parent link="base_link"/>
+        <child link="right_rear_wheel"/>
+        <origin xyz="-0.05 -0.058 0.025" rpy="${pi/2} 0.0 0.0"/>
+        <axis xyz="0.0 0.0 -1.0"/>
+    </joint>
+    <link name="right_rear_wheel">
         <visual>
             <geometry>
@@ -64,72 +147,6 @@
         </xacro:inertial_cylinder>
    </link>
-   <!-- LEFT REAR WHEEL LINK -->
-    <joint name="left_rear_wheel_joint" type="fixed">
-        <parent link="base_link"/>
-        <child link="left_rear_wheel"/>
-        <origin xyz="-0.05 0.058 0.025" rpy="-${pi/2} 0.0 0.0"/>
-        <axis xyz="0.0 0.0 1.0"/>
-    </joint>
-   <link name="left_rear_wheel">
-        <visual>
-            <geometry>
-                <cylinder radius="0.048" length="0.019"/>
-                <material name="blue"/>
-            </geometry>
-        </visual>
-        <collision>
-            <geometry>
-                <cylinder radius="0.048" length="0.019"/>
-            </geometry>
-        </collision>
-        <xacro:inertial_cylinder mass="0.1" length="0.019" radius="0.048">
-            <origin xyz="0 0 0" rpy="0 0 0" />
-        </xacro:inertial_cylinder>
-   </link>
-    <!-- RIGHT FRONT WHEEL LINK -->
-    <joint name="right_front_wheel_joint" type="fixed">
-        <parent link="base_link"/>
-        <child link="right_front_wheel"/>
-        <origin xyz="0.05 -0.058 0.025" rpy="${pi/2} 0.0 0.0"/>
-        <axis xyz="0.0 0.0 -1.0"/>
-    </joint>
-   <link name="right_front_wheel">
-        <visual>
-            <geometry>
-                <cylinder radius="0.048" length="0.019"/>
-                <material name="blue"/>
-            </geometry>
-        </visual>
-        <collision>
-            <geometry>
-                <cylinder radius="0.048" length="0.019"/>
-            </geometry>
-        </collision>
-        <xacro:inertial_cylinder mass="0.1" length="0.019" radius="0.048">
-            <origin xyz="0 0 0" rpy="0 0 0" />
-        </xacro:inertial_cylinder>
-   </link>
-   <!-- RIGHT REAR WHEEL LINK -->
-    <joint name="right_rear_wheel_joint" type="continuous">
-        <parent link="base_link"/>
-        <child link="right_rear_wheel"/>
-        <origin xyz="-0.05 -0.058 0.025" rpy="${pi/2} 0.0 0.0"/>
-        <axis xyz="0.0 0.0 -1.0"/>
-    </joint>
-   <link name="right_rear_wheel">
-        <visual>
-            <geometry>
-                <cylinder radius="0.048" length="0.019"/>
-                <material name="blue"/>
-            </geometry>
-        </visual>
-        <collision>
-            <geometry>
-                <cylinder radius="0.048" length="0.019"/>
-            </geometry>
-        </collision>
-        <xacro:inertial_cylinder mass="0.1" length="0.019" radius="0.048">
-            <origin xyz="0 0 0" rpy="0 0 0" />
-        </xacro:inertial_cylinder>
-   </link>
+    <gazebo reference="right_rear_wheel">
+        <material>Gazebo/Blue</material>
+    </gazebo>
 </robot>

Commit message: Add files to be used for actual robot

File: description/robot.urdf.xacro (robot description, xacro)
@@ -1,4 +1,5 @@
 <?xml version="1.0"?>
 <robot xmlns:xacro="http://www.ros.org/wiki/xacro"  name="robot">
+    <xacro:arg name="sim_mode" default="false" />
     <xacro:include filename="robot_core.xacro"/>
     <!-- <xacro:include filename="gazebo_control.xacro" /> -->

File: description/robot_core.xacro (robot description, xacro)
@@ -60,5 +60,5 @@
         <collision>
             <geometry>
-                <cylinder radius="0.048" length="0.019"/>
+                <sphere radius="0.048" />
             </geometry>
         </collision>
@@ -69,4 +69,6 @@
     <gazebo reference="left_front_wheel">
         <material>Gazebo/Blue</material>
+        <mu1 value="1.0"/>
+        <mu2 value="0.001" />
     </gazebo>
     <!-- LEFT REAR WHEEL LINK -->
@@ -86,5 +88,5 @@
         <collision>
             <geometry>
-                <cylinder radius="0.048" length="0.019"/>
+                <sphere radius="0.048"/>
             </geometry>
         </collision>
@@ -95,8 +97,9 @@
     <gazebo reference="left_rear_wheel">
         <material>Gazebo/Blue</material>
-        <mu1 value="0.001"/>
+        <mu1 value="1.0"/>
+        <mu2 value="0.001" />
     </gazebo>
     <!-- RIGHT FRONT WHEEL LINK -->
-    <joint name="right_front_wheel_joint" type="fixed">
+    <joint name="right_front_wheel_joint" type="continuous">
         <parent link="base_link"/>
         <child link="right_front_wheel"/>
@@ -113,5 +116,5 @@
         <collision>
             <geometry>
-                <cylinder radius="0.048" length="0.019"/>
+                <sphere radius="0.048" />
             </geometry>
         </collision>
@@ -122,8 +125,9 @@
     <gazebo reference="right_front_wheel">
         <material>Gazebo/Blue</material>
-        <mu1 value="0.001"/>
+        <mu1 value="1.0"/>
+        <mu2 value="0.001" />
     </gazebo>
    <!-- RIGHT REAR WHEEL LINK -->
-    <joint name="right_rear_wheel_joint" type="continuous">
+    <joint name="right_rear_wheel_joint" type="fixed">
         <parent link="base_link"/>
         <child link="right_rear_wheel"/>
@@ -140,5 +144,5 @@
         <collision>
             <geometry>
-                <cylinder radius="0.048" length="0.019"/>
+                <sphere radius="0.048" />
             </geometry>
         </collision>
@@ -149,4 +153,6 @@
     <gazebo reference="right_rear_wheel">
         <material>Gazebo/Blue</material>
+        <mu1 value="1.0"/>
+        <mu2 value="0.001" />
     </gazebo>
 </robot>

File: description/ros2_control.xacro (robot description, xacro)
@@ -1,28 +1,55 @@
 <?xml version="1.0"?>
 <robot xmlns:xacro="http://www.ros.org/wiki/xacro"  name="robot">
-    <ros2_control name="GazeboSystem" type="system">
-        <hardware>
-            <plugin>gazebo_ros2_control/GazeboSystem</plugin>
-        </hardware>
-        <joint name="left_front_wheel_joint">
-            <command_interface name="velocity">
-                <param name="min">-10</param>
-                <param name="max">10</param>
-            </command_interface>
-            <state_interface name="velocity" />
-            <state_interface name="position" />
-        </joint>
-        <joint name="right_rear_wheel_joint">
-            <command_interface name="velocity">
-                <param name="min">-10</param>
-                <param name="max">10</param>
-            </command_interface>
-            <state_interface name="velocity" />
-            <state_interface name="position" />
-        </joint>
-    </ros2_control>
+    <xacro:unless value="$(arg sim_mode)">
+        <ros2_control name="RealRobot" type="system">
+            <hardware>
+                <!-- TODO: Change to actual plugin once written -->
+                <plugin>gazebo_ros2_control/GazeboSystem</plugin>
+            </hardware>
+            <joint name="left_front_wheel_joint">
+                <command_interface name="velocity">
+                    <param name="min">-10</param>
+                    <param name="max">10</param>
+                </command_interface>
+                <state_interface name="velocity" />
+                <state_interface name="position" />
+            </joint>
+            <joint name="right_rear_wheel_joint">
+                <command_interface name="velocity">
+                    <param name="min">-10</param>
+                    <param name="max">10</param>
+                </command_interface>
+                <state_interface name="velocity" />
+                <state_interface name="position" />
+            </joint>
+        </ros2_control>
+    </xacro:unless>
+    <xacro:if value="$(arg sim_mode)">
+        <ros2_control name="GazeboSystem" type="system">
+            <hardware>
+                <plugin>gazebo_ros2_control/GazeboSystem</plugin>
+            </hardware>
+            <joint name="left_front_wheel_joint">
+                <command_interface name="velocity">
+                    <param name="min">-10</param>
+                    <param name="max">10</param>
+                </command_interface>
+                <state_interface name="velocity" />
+                <state_interface name="position" />
+            </joint>
+            <joint name="right_rear_wheel_joint">
+                <command_interface name="velocity">
+                    <param name="min">-10</param>
+                    <param name="max">10</param>
+                </command_interface>
+                <state_interface name="velocity" />
+                <state_interface name="position" />
+            </joint>
+        </ros2_control>
+    </xacro:if>
     <gazebo>
         <plugin name="gazebo_ros2_control" filename="libgazebo_ros2_control.so">
             <parameters>$(find mini_ocebot)/config/my_controllers.yaml</parameters>
+            <parameters>$(find mini_ocebot)/config/gaz_ros2_ctl_use_sim_time.yaml</parameters>
         </plugin>
     </gazebo>
