Commit message: Add 4 wheel differential drive control

File: description/robot_core.xacro (robot description, xacro)
@@ -69,9 +69,9 @@
     <gazebo reference="left_front_wheel">
         <material>Gazebo/Blue</material>
-        <mu1 value="1.0"/>
-        <mu2 value="0.001" />
+        <mu1 value="0.4"/>
+        <mu2 value="0.6" />
     </gazebo>
     <!-- LEFT REAR WHEEL LINK -->
-    <joint name="left_rear_wheel_joint" type="fixed">
+    <joint name="left_rear_wheel_joint" type="continuous">
         <parent link="base_link"/>
         <child link="left_rear_wheel"/>
@@ -97,6 +97,6 @@
     <gazebo reference="left_rear_wheel">
         <material>Gazebo/Blue</material>
-        <mu1 value="1.0"/>
-        <mu2 value="0.001" />
+        <mu1 value="0.4"/>
+        <mu2 value="0.6" />
     </gazebo>
     <!-- RIGHT FRONT WHEEL LINK -->
@@ -125,9 +125,9 @@
     <gazebo reference="right_front_wheel">
         <material>Gazebo/Blue</material>
-        <mu1 value="1.0"/>
-        <mu2 value="0.001" />
+        <mu1 value="0.4"/>
+        <mu2 value="0.6" />
     </gazebo>
    <!-- RIGHT REAR WHEEL LINK -->
-    <joint name="right_rear_wheel_joint" type="fixed">
+    <joint name="right_rear_wheel_joint" type="continuous">
         <parent link="base_link"/>
         <child link="right_rear_wheel"/>
@@ -153,6 +153,6 @@
     <gazebo reference="right_rear_wheel">
         <material>Gazebo/Blue</material>
-        <mu1 value="1.0"/>
-        <mu2 value="0.001" />
+        <mu1 value="0.4"/>
+        <mu2 value="0.6" />
     </gazebo>
 </robot>

File: description/ros2_control.xacro (robot description, xacro)
@@ -38,4 +38,20 @@
                 <state_interface name="position" />
             </joint>
+            <joint name="left_rear_wheel_joint">
+                <command_interface name="velocity">
+                    <param name="min">-10</param>
+                    <param name="max">10</param>
+                </command_interface>
+                <state_interface name="velocity" />
+                <state_interface name="position" />
+            </joint>
+            <joint name="right_front_wheel_joint">
+                <command_interface name="velocity">
+                    <param name="min">-10</param>
+                    <param name="max">10</param>
+                </command_interface>
+                <state_interface name="velocity" />
+                <state_interface name="position" />
+            </joint>
             <joint name="right_rear_wheel_joint">
                 <command_interface name="velocity">
